Commit message: Remove outdated world files for TurtleBot3 DQN stages 1 to 4 to streamline simulation environment.

File: src/amar_description/urdf/turtlebot3_burger_cam.urdf.xacro (robot description, xacro)
@@ -1,5 +1,5 @@
 <?xml version="1.0" ?>
 <robot name="turtlebot3_burger_cam"
-  xmlns:xacro="http://ros.org/wiki/xacro">
+  xmlns:xacro="http://ros.org">
   <material name="black">
       <color rgba="0.0 0.0 0.0 1.0"/>
@@ -36,24 +36,29 @@
     <parent link="base_footprint"/>
     <child link="base_link"/>
-    <origin xyz="0.0 0.0 0.010" rpy="0 0 0"/>
+    <!-- Z origin shifted up from 0.010 to 0.050 -->
+    <origin xyz="0.0 0.0 0.050" rpy="0 0 0"/>
   </joint>
   <link name="base_link">
     <visual>
-      <origin xyz="-0.032 0 0.0" rpy="0 0 0"/>
+      <!-- X position scaled from -0.032 to -0.160 -->
+      <origin xyz="-0.160 0 0.0" rpy="0 0 0"/>
       <geometry>
-        <mesh filename="file://$(find amar_description)/models/turtlebot3_common/meshes/bases/burger_base.stl" scale="0.001 0.001 0.001"/>
+        <!-- Mesh visual scale factor increased from 0.001 to 0.005 -->
+        <mesh filename="file://$(find amar_description)/models/turtlebot3_common/meshes/bases/burger_base.stl" scale="0.005 0.005 0.005"/>
       </geometry>
       <material name="light_black"/>
     </visual>
     <collision>
-      <origin xyz="-0.032 0 0.070" rpy="0 0 0"/>
+      <!-- Collision origin box extents scaled 5x -->
+      <origin xyz="-0.160 0 0.350" rpy="0 0 0"/>
       <geometry>
-        <box size="0.140 0.140 0.143"/>
+        <box size="0.700 0.700 0.715"/>
       </geometry>
     </collision>
     <inertial>
       <origin xyz="0 0 0" rpy="0 0 0"/>
-      <mass value="8.2573504e-01"/>
-      <inertia ixx="2.2124416e-03" ixy="-1.2294101e-05" ixz="3.4938785e-05" iyy="2.1193702e-03" iyz="-5.0120904e-06" izz="2.0064271e-03" />
+      <!-- Mass scaled realistically for stability (~15x) -->
+      <mass value="12.38"/>
+      <inertia ixx="3.31e-02" ixy="-1.84e-04" ixz="5.24e-04" iyy="3.17e-02" iyz="-7.51e-05" izz="3.00e-02" />
     </inertial>
   </link>
@@ -61,5 +66,6 @@
     <parent link="base_link"/>
     <child link="wheel_left_link"/>
-    <origin xyz="0.0 0.08 0.023" rpy="-1.57 0 0"/>
+    <!-- Joint attachment coordinates scaled 5x -->
+    <origin xyz="0.0 0.400 0.115" rpy="-1.57 0 0"/>
     <axis xyz="0 0 1"/>
   </joint>
@@ -68,5 +74,5 @@
       <origin xyz="0 0 0" rpy="1.57 0 0"/>
       <geometry>
-        <mesh filename="file://$(find amar_description)/models/turtlebot3_common/meshes/wheels/left_tire.stl" scale="0.001 0.001 0.001"/>
+        <mesh filename="file://$(find amar_description)/models/turtlebot3_common/meshes/wheels/left_tire.stl" scale="0.005 0.005 0.005"/>
       </geometry>
       <material name="dark"/>
@@ -75,11 +81,12 @@
       <origin xyz="0 0 0" rpy="0 0 0"/>
       <geometry>
-        <cylinder length="0.018" radius="0.033"/>
+        <!-- Cylinder metrics: length 0.09, radius 0.165 -->
+        <cylinder length="0.090" radius="0.165"/>
       </geometry>
     </collision>
     <inertial>
       <origin xyz="0 0 0" />
-      <mass value="2.8498940e-02" />
-      <inertia ixx="1.1175580e-05" ixy="-4.2369783e-11" ixz="-5.9381719e-09" iyy="1.1192413e-05" iyz="-1.4400107e-11" izz="2.0712558e-05" />
+      <mass value="0.427" />
+      <inertia ixx="1.67e-04" ixy="-6.35e-10" ixz="-8.90e-08" iyy="1.67e-04" iyz="-2.16e-10" izz="3.10e-04" />
     </inertial>
   </link>
@@ -87,5 +94,6 @@
     <parent link="base_link"/>
     <child link="wheel_right_link"/>
-    <origin xyz="0.0 -0.080 0.023" rpy="-1.57 0 0"/>
+    <!-- Joint attachment coordinates scaled 5x -->
+    <origin xyz="0.0 -0.400 0.115" rpy="-1.57 0 0"/>
     <axis xyz="0 0 1"/>
   </joint>
@@ -94,5 +102,5 @@
       <origin xyz="0 0 0" rpy="1.57 0 0"/>
       <geometry>
-        <mesh filename="file://$(find amar_description)/models/turtlebot3_common/meshes/wheels/right_tire.stl" scale="0.001 0.001 0.001"/>
+        <mesh filename="file://$(find amar_description)/models/turtlebot3_common/meshes/wheels/right_tire.stl" scale="0.005 0.005 0.005"/>
       </geometry>
       <material name="dark"/>
@@ -101,11 +109,11 @@
       <origin xyz="0 0 0" rpy="0 0 0"/>
       <geometry>
-        <cylinder length="0.018" radius="0.033"/>
+        <cylinder length="0.090" radius="0.165"/>
       </geometry>
     </collision>
     <inertial>
       <origin xyz="0 0 0" />
-      <mass value="2.8498940e-02" />
-      <inertia ixx="1.1175580e-05" ixy="-4.2369783e-11" ixz="-5.9381719e-09" iyy="1.1192413e-05" iyz="-1.4400107e-11" izz="2.0712558e-05" />
+      <mass value="0.427" />
+      <inertia ixx="1.67e-04" ixy="-6.35e-10" ixz="-8.90e-08" iyy="1.67e-04" iyz="-2.16e-10" izz="3.10e-04" />
     </inertial>
   </link>
@@ -113,17 +121,18 @@
     <parent link="base_link"/>
     <child link="caster_back_link"/>
-    <origin xyz="-0.081 0 -0.004" rpy="-1.57 0 0"/>
+    <!-- Coordinates scaled 5x -->
+    <origin xyz="-0.405 0 -0.020" rpy="-1.57 0 0"/>
   </joint>
   <link name="caster_back_link">
     <collision>
-      <origin xyz="0 0.001 0" rpy="0 0 0"/>
+      <origin xyz="0 0.005 0" rpy="0 0 0"/>
       <geometry>
-        <box size="0.030 0.009 0.020"/>
+        <box size="0.150 0.045 0.100"/>
       </geometry>
     </collision>
     <inertial>
       <origin xyz="0 0 0" />
-      <mass value="0.005" />
-      <inertia ixx="0.001" ixy="0.0" ixz="0.0" iyy="0.001" iyz="0.0" izz="0.001" />
+      <mass value="0.075" />
+      <inertia ixx="0.015" ixy="0.0" ixz="0.0" iyy="0.015" iyz="0.0" izz="0.015" />
     </inertial>
   </link>
@@ -131,5 +140,5 @@
     <parent link="base_link"/>
     <child link="imu_link"/>
-    <origin xyz="-0.032 0 0.068" rpy="0 0 0"/>
+    <origin xyz="-0.160 0 0.340" rpy="0 0 0"/>
   </joint>
   <link name="imu_link"/>
@@ -137,5 +146,5 @@
     <parent link="base_link"/>
     <child link="base_scan"/>
-    <origin xyz="-0.032 0 0.172" rpy="0 0 0"/>
+    <origin xyz="-0.160 0 0.860" rpy="0 0 0"/>
   </joint>
   <link name="base_scan">
@@ -143,22 +152,22 @@
       <origin xyz="0 0 0.0" rpy="0 0 0"/>
       <geometry>
-        <mesh filename="file://$(find amar_description)/models/turtlebot3_common/meshes/sensors/lds.stl" scale="0.001 0.001 0.001"/>
+        <mesh filename="file://$(find amar_description)/models/turtlebot3_common/meshes/sensors/lds.stl" scale="0.005 0.005 0.005"/>
       </geometry>
       <material name="dark"/>
     </visual>
     <collision>
-      <origin xyz="0.015 0 -0.0065" rpy="0 0 0"/>
+      <origin xyz="0.075 0 -0.0325" rpy="0 0 0"/>
       <geometry>
-        <cylinder length="0.0315" radius="0.055"/>
+        <cylinder length="0.1575" radius="0.275"/>
       </geometry>
     </collision>
     <inertial>
-      <mass value="0.114" />
+      <mass value="1.71" />
       <origin xyz="0 0 0" />
-      <inertia ixx="0.001" ixy="0.0" ixz="0.0" iyy="0.001" iyz="0.0" izz="0.001" />
+      <inertia ixx="0.015" ixy="0.0" ixz="0.0" iyy="0.015" iyz="0.0" izz="0.015" />
     </inertial>
   </link>
   <joint name="camera_joint" type="fixed">
-    <origin xyz="0.040 -0.000 0.110" rpy="0 0 0"/>
+    <origin xyz="0.200 -0.000 0.550" rpy="0 0 0"/>
     <parent link="base_link"/>
     <child link="camera_link"/>
@@ -166,12 +175,12 @@
   <link name="camera_link">
     <collision>
-      <origin xyz="0.005 0.000 0.013" rpy="0 0 0"/>
+      <origin xyz="0.025 0.000 0.065" rpy="0 0 0"/>
       <geometry>
-        <box size="0.015 0.030 0.027"/>
+        <box size="0.075 0.150 0.135"/>
       </geometry>
     </collision>
   </link>
   <joint name="camera_rgb_joint" type="fixed">
-    <origin xyz="0.003 0.000 0.009" rpy="0 0 0"/>
+    <origin xyz="0.015 0.000 0.045" rpy="0 0 0"/>
     <parent link="camera_link"/>
     <child link="camera_rgb_frame"/>

Commit message: Add TurtleBot3 Burger with Camera Model and Navigation Parameters
- Created URDF model for TurtleBot3 Burger with camera integration, including links for wheels, IMU, and LIDAR.
- Added SDF model for simulation, defining physical properties, sensors, and joints for the TurtleBot3 Burger.
- Introduced navigation parameters in YAML format for AMCL, BT Navigator, Docking Server, Controller Server, and Costmaps to facilitate robot navigation and obstacle avoidance.

File: src/amar_description/urdf/turtlebot3_burger_cam.urdf.xacro (robot description, xacro)
@@ -1,5 +1,5 @@
 <?xml version="1.0" ?>
 <robot name="turtlebot3_burger_cam"
-  xmlns:xacro="http://ros.org">
+  xmlns:xacro="http://ros.org/wiki/xacro">
   <material name="black">
       <color rgba="0.0 0.0 0.0 1.0"/>
@@ -36,29 +36,24 @@
     <parent link="base_footprint"/>
     <child link="base_link"/>
-    <!-- Z origin shifted up from 0.010 to 0.050 -->
-    <origin xyz="0.0 0.0 0.050" rpy="0 0 0"/>
+    <origin xyz="0.0 0.0 0.010" rpy="0 0 0"/>
   </joint>
   <link name="base_link">
     <visual>
-      <!-- X position scaled from -0.032 to -0.160 -->
-      <origin xyz="-0.160 0 0.0" rpy="0 0 0"/>
+      <origin xyz="-0.032 0 0.0" rpy="0 0 0"/>
       <geometry>
-        <!-- Mesh visual scale factor increased from 0.001 to 0.005 -->
-        <mesh filename="file://$(find amar_description)/models/turtlebot3_common/meshes/bases/burger_base.stl" scale="0.005 0.005 0.005"/>
+        <mesh filename="file://$(find amar_description)/models/turtlebot3_common/meshes/bases/burger_base.stl" scale="0.001 0.001 0.001"/>
       </geometry>
       <material name="light_black"/>
     </visual>
     <collision>
-      <!-- Collision origin box extents scaled 5x -->
-      <origin xyz="-0.160 0 0.350" rpy="0 0 0"/>
+      <origin xyz="-0.032 0 0.070" rpy="0 0 0"/>
       <geometry>
-        <box size="0.700 0.700 0.715"/>
+        <box size="0.140 0.140 0.143"/>
       </geometry>
     </collision>
     <inertial>
       <origin xyz="0 0 0" rpy="0 0 0"/>
-      <!-- Mass scaled realistically for stability (~15x) -->
-      <mass value="12.38"/>
-      <inertia ixx="3.31e-02" ixy="-1.84e-04" ixz="5.24e-04" iyy="3.17e-02" iyz="-7.51e-05" izz="3.00e-02" />
+      <mass value="8.2573504e-01"/>
+      <inertia ixx="2.2124416e-03" ixy="-1.2294101e-05" ixz="3.4938785e-05" iyy="2.1193702e-03" iyz="-5.0120904e-06" izz="2.0064271e-03" />
     </inertial>
   </link>
@@ -66,6 +61,5 @@
     <parent link="base_link"/>
     <child link="wheel_left_link"/>
-    <!-- Joint attachment coordinates scaled 5x -->
-    <origin xyz="0.0 0.400 0.115" rpy="-1.57 0 0"/>
+    <origin xyz="0.0 0.08 0.023" rpy="-1.57 0 0"/>
     <axis xyz="0 0 1"/>
   </joint>
@@ -74,5 +68,5 @@
       <origin xyz="0 0 0" rpy="1.57 0 0"/>
       <geometry>
-        <mesh filename="file://$(find amar_description)/models/turtlebot3_common/meshes/wheels/left_tire.stl" scale="0.005 0.005 0.005"/>
+        <mesh filename="file://$(find amar_description)/models/turtlebot3_common/meshes/wheels/left_tire.stl" scale="0.001 0.001 0.001"/>
       </geometry>
       <material name="dark"/>
@@ -81,12 +75,11 @@
       <origin xyz="0 0 0" rpy="0 0 0"/>
       <geometry>
-        <!-- Cylinder metrics: length 0.09, radius 0.165 -->
-        <cylinder length="0.090" radius="0.165"/>
+        <cylinder length="0.018" radius="0.033"/>
       </geometry>
     </collision>
     <inertial>
       <origin xyz="0 0 0" />
-      <mass value="0.427" />
-      <inertia ixx="1.67e-04" ixy="-6.35e-10" ixz="-8.90e-08" iyy="1.67e-04" iyz="-2.16e-10" izz="3.10e-04" />
+      <mass value="2.8498940e-02" />
+      <inertia ixx="1.1175580e-05" ixy="-4.2369783e-11" ixz="-5.9381719e-09" iyy="1.1192413e-05" iyz="-1.4400107e-11" izz="2.0712558e-05" />
     </inertial>
   </link>
@@ -94,6 +87,5 @@
     <parent link="base_link"/>
     <child link="wheel_right_link"/>
-    <!-- Joint attachment coordinates scaled 5x -->
-    <origin xyz="0.0 -0.400 0.115" rpy="-1.57 0 0"/>
+    <origin xyz="0.0 -0.080 0.023" rpy="-1.57 0 0"/>
     <axis xyz="0 0 1"/>
   </joint>
@@ -102,5 +94,5 @@
       <origin xyz="0 0 0" rpy="1.57 0 0"/>
       <geometry>
-        <mesh filename="file://$(find amar_description)/models/turtlebot3_common/meshes/wheels/right_tire.stl" scale="0.005 0.005 0.005"/>
+        <mesh filename="file://$(find amar_description)/models/turtlebot3_common/meshes/wheels/right_tire.stl" scale="0.001 0.001 0.001"/>
       </geometry>
       <material name="dark"/>
@@ -109,11 +101,11 @@
       <origin xyz="0 0 0" rpy="0 0 0"/>
       <geometry>
-        <cylinder length="0.090" radius="0.165"/>
+        <cylinder length="0.018" radius="0.033"/>
       </geometry>
     </collision>
     <inertial>
       <origin xyz="0 0 0" />
-      <mass value="0.427" />
-      <inertia ixx="1.67e-04" ixy="-6.35e-10" ixz="-8.90e-08" iyy="1.67e-04" iyz="-2.16e-10" izz="3.10e-04" />
+      <mass value="2.8498940e-02" />
+      <inertia ixx="1.1175580e-05" ixy="-4.2369783e-11" ixz="-5.9381719e-09" iyy="1.1192413e-05" iyz="-1.4400107e-11" izz="2.0712558e-05" />
     </inertial>
   </link>
@@ -121,18 +113,17 @@
     <parent link="base_link"/>
     <child link="caster_back_link"/>
-    <!-- Coordinates scaled 5x -->
-    <origin xyz="-0.405 0 -0.020" rpy="-1.57 0 0"/>
+    <origin xyz="-0.081 0 -0.004" rpy="-1.57 0 0"/>
   </joint>
   <link name="caster_back_link">
     <collision>
-      <origin xyz="0 0.005 0" rpy="0 0 0"/>
+      <origin xyz="0 0.001 0" rpy="0 0 0"/>
       <geometry>
-        <box size="0.150 0.045 0.100"/>
+        <box size="0.030 0.009 0.020"/>
       </geometry>
     </collision>
     <inertial>
       <origin xyz="0 0 0" />
-      <mass value="0.075" />
-      <inertia ixx="0.015" ixy="0.0" ixz="0.0" iyy="0.015" iyz="0.0" izz="0.015" />
+      <mass value="0.005" />
+      <inertia ixx="0.001" ixy="0.0" ixz="0.0" iyy="0.001" iyz="0.0" izz="0.001" />
     </inertial>
   </link>
@@ -140,5 +131,5 @@
     <parent link="base_link"/>
     <child link="imu_link"/>
-    <origin xyz="-0.160 0 0.340" rpy="0 0 0"/>
+    <origin xyz="-0.032 0 0.068" rpy="0 0 0"/>
   </joint>
   <link name="imu_link"/>
@@ -146,5 +137,5 @@
     <parent link="base_link"/>
     <child link="base_scan"/>
-    <origin xyz="-0.160 0 0.860" rpy="0 0 0"/>
+    <origin xyz="-0.032 0 0.172" rpy="0 0 0"/>
   </joint>
   <link name="base_scan">
@@ -152,22 +143,22 @@
       <origin xyz="0 0 0.0" rpy="0 0 0"/>
       <geometry>
-        <mesh filename="file://$(find amar_description)/models/turtlebot3_common/meshes/sensors/lds.stl" scale="0.005 0.005 0.005"/>
+        <mesh filename="file://$(find amar_description)/models/turtlebot3_common/meshes/sensors/lds.stl" scale="0.001 0.001 0.001"/>
       </geometry>
       <material name="dark"/>
     </visual>
     <collision>
-      <origin xyz="0.075 0 -0.0325" rpy="0 0 0"/>
+      <origin xyz="0.015 0 -0.0065" rpy="0 0 0"/>
       <geometry>
-        <cylinder length="0.1575" radius="0.275"/>
+        <cylinder length="0.0315" radius="0.055"/>
       </geometry>
     </collision>
     <inertial>
-      <mass value="1.71" />
+      <mass value="0.114" />
       <origin xyz="0 0 0" />
-      <inertia ixx="0.015" ixy="0.0" ixz="0.0" iyy="0.015" iyz="0.0" izz="0.015" />
+      <inertia ixx="0.001" ixy="0.0" ixz="0.0" iyy="0.001" iyz="0.0" izz="0.001" />
     </inertial>
   </link>
   <joint name="camera_joint" type="fixed">
-    <origin xyz="0.200 -0.000 0.550" rpy="0 0 0"/>
+    <origin xyz="0.040 -0.000 0.110" rpy="0 0 0"/>
     <parent link="base_link"/>
     <child link="camera_link"/>
@@ -175,12 +166,12 @@
   <link name="camera_link">
     <collision>
-      <origin xyz="0.025 0.000 0.065" rpy="0 0 0"/>
+      <origin xyz="0.005 0.000 0.013" rpy="0 0 0"/>
       <geometry>
-        <box size="0.075 0.150 0.135"/>
+        <box size="0.015 0.030 0.027"/>
       </geometry>
     </collision>
   </link>
   <joint name="camera_rgb_joint" type="fixed">
-    <origin xyz="0.015 0.000 0.045" rpy="0 0 0"/>
+    <origin xyz="0.003 0.000 0.009" rpy="0 0 0"/>
     <parent link="camera_link"/>
     <child link="camera_rgb_frame"/>
